File: SashSense_node2/Firefly_pcb2.kicad_pcb (KiCad board)
At the start: 2 copper layers, 500 x 500 mm, 67 parts, among them J1 REGULATED 3.3V IN, J2 UART / BOOT SERVICE, Q1 MMBT3904LT1G, SW1 RESET, SW2 BOOT, U1 ESP32-S3-WROOM-1-N8, U2 VL53L1CXV0FY/1, U3 AMG8833

Commit message: Trim Firefly presence board to 160 x 60 mm
Cut the unused area from the provisional 500 x 500 mm outline. Placement
and routing are unchanged; the support grid becomes four corner M3 holes.
Refresh the native CAD, KiCad check reports, plots, previews and docs.
Parts:
- removed H10, H11, H12, H13, H14, H15, H16, H17, H18, H19, H20, H21, H22, H23, H24, H25, H5, H6, H7, H8, H9: M3 SUPPORT - PROVISIONAL, SashSense:MountingHole_3.2mm_M3
- moved H3 244.2 mm to (35.0, 80.0)
- moved H4 214.8 mm to (185.0, 80.0)
- moved H2 30.4 mm to (185.0, 30.0)
- moved FID2 12.8 mm to (176.0, 40.0)
- moved H1 5.00 mm to (35.0, 30.0)
Routing:
- net /GND: vias 191 -> 211
Other:
- board size 500 x 500 mm -> 160 x 60 mm
- board text added: "Firefly_pcb2 P2 - BOTTOM | 160 x 60 mm"
- board text removed: "500.00 x 500.00 mm | 2 layers | 1.6 mm nominal | M3 support grid PROVISIONAL"
- board text removed: "Firefly_pcb2 P2 - BOTTOM"
