File: SashSense_node1.kicad_pcb (KiCad board)
At the start: 2 copper layers, 50 x 50 mm, 29 parts, among them J1 Conn_01x02_Pin, J2 USB_C_Receptacle_USB2.0_16P, SW1 reset, SW2 boot, U1 ESP32-WROOM-32E, U2 SHT31-DIS, U3 AMS1117-3.3, U4 CP2102N-Axx-xQFN24, U5 VL53L0CXV0DH1

Commit message: Switch node 1 to VL53L1X and fix its rule-check findings
Replace the VL53L0X symbol on U5 with the pin-compatible VL53L1X; the board
already used the VL53L1x footprint. Move SCL and the parallel +5V run off the
board edge, join the split top ground pour with GND vias and short bottom
jumpers, rotate C5 so its ground pad reaches the pour, and fix two silkscreen
warnings. Refresh node 1 reports, PDF, SVG and preview images.
Parts:
- U5: value VL53L0CXV0DH1 -> VL53L1CXV0FY1
- turned C5 to 180 degrees
Routing:
- net GND: track 7.11 -> 30.2 mm, vias 0 -> 16
- net /SCL: track 208.4 -> 207.7 mm
Other:
- board text added: "VL53L1CXV0FY1"
- board text removed: "VL53L0CXV0DH1"
Changed lines of the file:
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@@
 			)
 		)
-		(property "Value" "VL53L0CXV0DH1"
+		(property "Value" "VL53L1CXV0FY1"
 			(at 0.26 -5.46 180)
 			(layer "F.Fab")
@@
 			)
 		)
-		(property "Datasheet" "https://www.st.com/resource/en/datasheet/vl53l0x.pdf"
+		(property "Datasheet" "https://www.st.com/resource/en/datasheet/vl53l1x.pdf"
 			(at 0 0 0)
 			(unlocked yes)
@@
 			)
 		)
-		(property "Description" "2m distance ranging ToF sensor, Optical LGA12"
+		(property "Description" "4m distance ranging ToF sensor, Optical LGA12"
 			(at 0 0 0)
 			(unlocked yes)
@@
 	(footprint "Capacitor_SMD:C_0603_1608Metric"
 		(layer "F.Cu")
-		(at 55.5 132)
+		(at 55.5 132 180)
 		(descr "Capacitor SMD 0603 (1608 Metric), square (rectangular) end terminal, IPC-7351 nominal, (Body size source: IPC-SM-782 page 76, https://www.pcb-3d.com/wordpress/wp-content/uploads/ipc-sm-782a_amendment_1_and_2.pdf)")
 		(tags "capacitor")
 		(property "Reference" "C5"
-			(at 0 -1.43 0)
+			(at 0 -1.43 180)
 			(layer "F.SilkS")
 			(hide yes)
@@
 		)
 		(property "Value" "10uF"
-			(at 0 1.43 0)
+			(at 0 1.43 180)
 			(layer "F.Fab")
 			(hide yes)
@@
 		)
 		(property "Datasheet" ""
-			(at 0 0 0)
+			(at 0 0 180)
 			(layer "F.Fab")
 			(hide yes)
@@
 		)
 		(property "Description" "Unpolarized capacitor"
-			(at 0 0 0)
+			(at 0 0 180)
 			(layer "F.Fab")
 			(hide yes)
@@
 		)
 		(property "KiLib_Generator" "SMD_2terminal_chip_molded"
-			(at 0 0 0)
+			(at 0 0 180)
 			(layer "F.SilkS")
 			(hide yes)
@@
 		(duplicate_pad_numbers_are_jumpers no)
 		(fp_line
-			(start -0.14058 -0.51)
-			(end 0.14058 -0.51)
+			(start -0.14058 0.51)
+			(end 0.14058 0.51)
 			(stroke
 				(width 0.12)
@@
 		)
 		(fp_line
-			(start -0.14058 0.51)
-			(end 0.14058 0.51)
+			(start -0.14058 -0.51)
+			(end 0.14058 -0.51)
 			(stroke
 				(width 0.12)
@@
 		)
 		(fp_text user "${REFERENCE}"
-			(at 0 0 0)
+			(at 0 0 180)
 			(layer "F.Fab")
 			(effects
@@
 		)
 		(pad "1" smd roundrect
-			(at -0.775 0)
+			(at -0.775 0 180)
 			(size 0.9 0.95)
 			(layers "F.Cu" "F.Mask" "F.Paste")
@@
 		)
 		(pad "2" smd roundrect
-			(at 0.775 0)
+			(at 0.775 0 180)
 			(size 0.9 0.95)
 			(layers "F.Cu" "F.Mask" "F.Paste")
@@
 		(effects
 			(font
-				(size 0.7 0.7)
-				(thickness 0.1)
+				(size 0.8 0.8)
+				(thickness 0.12)
 			)
 			(justify left bottom)
 		)
 	)
-	(gr_text "VL53L0CXV0DH1"
+	(gr_text "VL53L1CXV0FY1"
 		(at 36.82 90.75 0)
 		(layer "F.SilkS")
@@
 	)
 	(gr_text "RESET"
-		(at 47 112.35 0)
+		(at 47.5 112.35 0)
 		(layer "F.SilkS")
 		(effects
@@
 		(net "GND")
 	)
+	(via
+		(at 52.251 100.5)
+		(size 0.6)
+		(drill 0.3)
+		(layers "F.Cu" "B.Cu")
+		(net "GND")
+	)
+	(via
+		(at 77.491 93.154)
+		(size 0.6)
+		(drill 0.3)
+		(layers "F.Cu" "B.Cu")
+		(net "GND")
+	)
+	(via
+		(at 69.463 116.91)
+		(size 0.6)
+		(drill 0.3)
+		(layers "F.Cu" "B.Cu")
+		(net "GND")
+	)
+	(via
+		(at 49.126 122.679)
+		(size 0.6)
+		(drill 0.3)
+		(layers "F.Cu" "B.Cu")
+		(net "GND")
+	)
+	(via
+		(at 52.853 102.722)
+		(size 0.6)
+		(drill 0.3)
+		(layers "F.Cu" "B.Cu")
+		(net "GND")
+	)
+	(via
+		(at 72.175 116.838)
+		(size 0.6)
+		(drill 0.3)
+		(layers "F.Cu" "B.Cu")
+		(net "GND")
+	)
+	(via
+		(at 52.251 91)
+		(size 0.6)
+		(drill 0.3)
+		(layers "F.Cu" "B.Cu")
+		(net "GND")
+	)
+	(via
+		(at 46.751 122.75)
+		(size 0.6)
+		(drill 0.3)
+		(layers "F.Cu" "B.Cu")
+		(net "GND")
+	)
+	(via
+		(at 44.3 91.925)
+		(size 0.6)
+		(drill 0.3)
+		(layers "F.Cu" "B.Cu")
+		(net "GND")
+	)
+	(via
+		(at 47.376 90.876)
+		(size 0.6)
+		(drill 0.3)
+		(layers "F.Cu" "B.Cu")
+		(net "GND")
+	)
+	(via
+		(at 72.175 121.338)
+		(size 0.6)
+		(drill 0.3)
+		(layers "F.Cu" "B.Cu")
+		(net "GND")
+	)
+	(via
+		(at 53.103 103.722)
+		(size 0.6)
+		(drill 0.3)
+		(layers "F.Cu" "B.Cu")
+		(net "GND")
+	)
+	(via
+		(at 80.001 90.75)
+		(size 0.6)
+		(drill 0.3)
+		(layers "F.Cu" "B.Cu")
+		(net "GND")
+	)
+	(via
+		(at 47.126 91.876)
+		(size 0.6)
+		(drill 0.3)
+		(layers "F.Cu" "B.Cu")
+		(net "GND")
+	)
+	(via
+		(at 70.626 122.929)
+		(size 0.6)
+		(drill 0.3)
+		(layers "F.Cu" "B.Cu")
+		(net "GND")
+	)
+	(via
+		(at 51.717 105.615)
+		(size 0.6)
+		(drill 0.3)
+		(layers "F.Cu" "B.Cu")
+		(net "GND")
+	)
+	(segment
+		(start 69.463 116.91)
+		(end 72.175 116.838)
+		(width 0.3)
+		(layer "B.Cu")
+		(net "GND")
+	)
+	(segment
+		(start 52.853 102.722)
+		(end 52.251 100.5)
+		(width 0.3)
+		(layer "B.Cu")
+		(net "GND")
+	)
+	(segment
+		(start 77.491 93.154)
+		(end 80.001 90.75)
+		(width 0.3)
+		(layer "B.Cu")
+		(net "GND")
+	)
+	(segment
+		(start 51.717 105.615)
+		(end 53.103 103.722)
+		(width 0.3)
+		(layer "B.Cu")
+		(net "GND")
+	)
+	(segment
+		(start 72.175 121.338)
+		(end 70.626 122.929)
+		(width 0.3)
+		(layer "B.Cu")
+		(net "GND")
+	)
+	(segment
+		(start 44.3 91.925)
+		(end 47.126 91.876)
+		(width 0.3)
+		(layer "B.Cu")
+		(net "GND")
+	)
+	(segment
+		(start 49.126 122.679)
+		(end 46.751 122.75)
+		(width 0.3)
+		(layer "B.Cu")
+		(net "GND")
+	)
+	(segment
+		(start 47.376 90.876)
+		(end 52.251 91)
+		(width 0.3)
+		(layer "B.Cu")
+		(net "GND")
+	)
 	(segment
 		(start 39.66 93.125)
@@
 	)
 	(segment
-		(start 84 96.431802)
+		(start 83.8 96.232)
 		(end 76.588198 89.02)
 		(width 0.25)
@@
 	)
 	(segment
-		(start 48 133)
-		(end 48.075 133.075)
-		(width 0.25)
-		(layer "F.Cu")
-		(net "/SCL")
-	)
-	(segment
 		(start 51.575 103.765)
 		(end 51.575 102.493198)
@@
 	)
 	(segment
-		(start 48.075 133.075)
-		(end 84 133.075)
+		(start 48 132.85)
+		(end 83.8 132.85)
 		(width 0.25)
 		(layer "F.Cu")
@@
 	)
 	(segment
-		(start 84 133.075)
-		(end 84 96.431802)
+		(start 83.8 132.85)
+		(end 83.8 96.232)
 		(width 0.25)
 		(layer "F.Cu")
@@
 	(segment
 		(start 48 121.575)
-		(end 48 133)
+		(end 48 132.85)
 		(width 0.25)
 		(layer "F.Cu")
@@
 	)
 	(segment
-		(start 82.6 132.5)
+		(start 82.6 132.25)
 		(end 82.6 130.4)
 		(width 0.5)
@@
 	)
 	(segment
-		(start 54.725 131)
-		(end 54.725 130.325)
+		(start 56.275 131)
+		(end 56.275 132)
 		(width 0.5)
 		(layer "F.Cu")
@@
 	(segment
 		(start 54.725 131)
-		(end 56.710828 131)
+		(end 54.725 130.325)
 		(width 0.5)
 		(layer "F.Cu")
@@
 	)
 	(segment
-		(start 54.725 131.2)
-		(end 54.725 131)
+		(start 57.961 132.25)
+		(end 82.6 132.25)
 		(width 0.5)
 		(layer "F.Cu")
@@
 	)
 	(segment
-		(start 58.210828 132.5)
-		(end 82.6 132.5)
+		(start 56.275 131)
+		(end 56.711 131)
 		(width 0.5)
 		(layer "F.Cu")
@@
 	)
 	(segment
-		(start 54.725 132)
-		(end 54.725 131.2)
+		(start 54.725 131)
+		(end 56.275 131)
 		(width 0.5)
 		(layer "F.Cu")
@@
 	(segment
 		(start 56.710828 131)
-		(end 58.210828 132.5)
+		(end 57.961 132.25)
 		(width 0.5)
 		(layer "F.Cu")
