File: SashSense_node1.kicad_sch (KiCad schematic)
At the start: 29 parts, among them J1 Conn_01x02_Pin, J2 USB_C_Receptacle_USB2.0_16P, SW1 reset, SW2 boot, U1 ESP32-WROOM-32E, U2 SHT31-DIS, U3 AMS1117-3.3, U4 CP2102N-Axx-xQFN24, U5 VL53L0CXV0DH1

Commit message: Switch node 1 to VL53L1X and fix its rule-check findings
Replace the VL53L0X symbol on U5 with the pin-compatible VL53L1X; the board
already used the VL53L1x footprint. Move SCL and the parallel +5V run off the
board edge, join the split top ground pour with GND vias and short bottom
jumpers, rotate C5 so its ground pad reaches the pour, and fix two silkscreen
warnings. Refresh node 1 reports, PDF, SVG and preview images.
Parts:
- U5: value VL53L0CXV0DH1 -> VL53L1CXV0FY1; symbol Sensor_Distance:VL53L0CXV0DH1 -> Sensor_Distance:VL53L1CXV0FY1
Changed lines of the file:
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@@
 	)
 	(symbol
-		(lib_id "Sensor_Distance:VL53L0CXV0DH1")
+		(lib_id "Sensor_Distance:VL53L1CXV0FY1")
 		(at 55.88 172.72 180)
 		(unit 1)
@@
 			)
 		)
-		(property "Value" "VL53L0CXV0DH1"
+		(property "Value" "VL53L1CXV0FY1"
 			(at 46.99 171.4501 0)
 			(show_name no)
@@
 			)
 		)
-		(property "Datasheet" "https://www.st.com/resource/en/datasheet/vl53l0x.pdf"
+		(property "Datasheet" "https://www.st.com/resource/en/datasheet/vl53l1x.pdf"
 			(at 53.34 172.72 0)
 			(hide yes)
@@
 			)
 		)
-		(property "Description" "2m distance ranging ToF sensor, Optical LGA12"
+		(property "Description" "4m distance ranging ToF sensor, Optical LGA12"
 			(at 55.88 172.72 0)
 			(hide yes)
